Commit message: new limo.urdf

File: limo_description/urdf/limo.urdf (robot description, URDF)
Before this commit: robot limo_ackerman, 13 links, 12 joints
Links:
- link base_link: geometry collision box size=0.13 0.12 0.1; visual mesh filename=package://Assets/O3DEScene/limo.fbx scale=1 1 1
- link front_left_wheel_link: geometry collision cylinder length=0.045 radius=0.045; visual mesh filename=package://Assets/O3DEScene/limoWheels.fbx
- link front_right_wheel_link: geometry collision cylinder length=0.045 radius=0.045; visual mesh filename=package://Assets/O3DEScene/limoWheels.fbx
- link rear_left_wheel_link: geometry collision cylinder length=0.045 radius=0.045; visual mesh filename=package://Assets/O3DEScene/limoWheels.fbx
- link rear_right_wheel_link: geometry collision cylinder length=0.045 radius=0.045; visual mesh filename=package://Assets/O3DEScene/limoWheels.fbx
